Commit message: README update

File: src/x500_description/urdf/x500.urdf (robot description, URDF)
Before this commit: robot x500, 9 links, 8 joints
Links:
- link lidar_2d_v2: geometry visual box size=0.001 0.001 0.001

Commit message: Tf fixing and readme

File: src/x500_description/urdf/x500.urdf (robot description, URDF)
Before this commit: robot x500, 9 links, 8 joints
Links:
- removed link lidar_2d_v2
- added link lidar_link/lidar_2d_v2; visual box size=0.001 0.001 0.001
Joints:
- joint lidar_2d_v2_joint: child lidar_2d_v2 -> lidar_link/lidar_2d_v2
