Commit message: lidar update

File: src/loki_config/urdf/loki.urdf (robot description, URDF)
Before this commit: robot drone, 2 links, 1 joints
Joints:
- joint base_to_lidar: origin xyz=-0.10 0.0 0.10 rpy=0 0 0 -> xyz=-0.10 0.0 0.10 rpy=0 0 3.1416

Commit message: loki urdf fix

File: src/loki_config/urdf/loki.urdf (robot description, URDF)
Before this commit: robot drone, 2 links, 1 joints
Joints:
- joint base_to_lidar: origin xyz=-0.10 0.0 0.10 rpy=0 0 3.1416 -> xyz=-0.10 0.0 0.10 rpy=0 0 0

Commit message: help

File: src/loki_config/urdf/loki.urdf (robot description, URDF)
Before this commit: robot drone, 2 links, 1 joints
Joints:
- joint base_to_lidar: origin xyz=-0.10 0.0 0.10 rpy=0 0 0 -> xyz=0 0 0.10 rpy=3.1416 0 0

Commit message: maybe fix

File: src/loki_config/urdf/loki.urdf (robot description, URDF)
Before this commit: robot drone, 2 links, 1 joints
Joints:
- joint base_to_lidar: origin xyz=0 0 0.10 rpy=3.1416 0 0 -> xyz=0 0 0.10 rpy=0 0 0
